File: Hardware/KiCad/Peripherals.kicad_sch (KiCad schematic)
At the start: 61 parts

Commit message: Added more footprints
Parts:
- C? (x4): footprint (none) -> Capacitor_SMD:C_0603_1608Metric
- C? (x9): footprint (none) -> Capacitor_SMD:C_0402_1005Metric
- D? (x2): footprint (none) -> LED_SMD:LED_0603_1608Metric
- FB? (x2): footprint (none) -> Inductor_SMD:L_0603_1608Metric
- R? (x2): footprint (none) -> Resistor_SMD:R_0402_1005Metric
- R? (x10): footprint Resistor_SMD:R_0603_1608Metric -> Resistor_SMD:R_0402_1005Metric
Changed lines of the file:
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@@
       (effects (font (size 1.27 1.27)) (justify left))
     )
-    (property "Footprint" "" (id 2) (at 146.685 50.8 0)
+    (property "Footprint" "Capacitor_SMD:C_0603_1608Metric" (id 2) (at 146.685 50.8 0)
       (effects (font (size 1.27 1.27)) hide)
     )
@@
     (property "Reference" "R?" (id 0) (at 85.725 160.02 90))
     (property "Value" "10k" (id 1) (at 85.725 161.925 90))
-    (property "Footprint" "" (id 2) (at 85.725 163.83 0)
+    (property "Footprint" "Resistor_SMD:R_0402_1005Metric" (id 2) (at 85.725 163.83 0)
       (effects (font (size 1.27 1.27)) hide)
     )
@@
       (effects (font (size 1.27 1.27)) (justify left))
     )
-    (property "Footprint" "" (id 2) (at 132.08 113.665 0)
+    (property "Footprint" "Capacitor_SMD:C_0402_1005Metric" (id 2) (at 132.08 113.665 0)
       (effects (font (size 1.27 1.27)) hide)
     )
@@
     (property "Reference" "FB?" (id 0) (at 53.975 22.86 90))
     (property "Value" "100@100MHz" (id 1) (at 53.975 24.765 90))
-    (property "Footprint" "" (id 2) (at 53.975 26.162 90)
+    (property "Footprint" "Inductor_SMD:L_0603_1608Metric" (id 2) (at 53.975 26.162 90)
       (effects (font (size 1.27 1.27)) hide)
     )
@@
     (property "Reference" "R?" (id 0) (at 203.835 95.885 0))
     (property "Value" "4k7" (id 1) (at 204.47 97.79 0))
-    (property "Footprint" "Resistor_SMD:R_0603_1608Metric" (id 2) (at 201.295 96.52 0)
+    (property "Footprint" "Resistor_SMD:R_0402_1005Metric" (id 2) (at 201.295 96.52 0)
       (effects (font (size 1.27 1.27)) hide)
     )
@@
     (property "Reference" "R?" (id 0) (at 178.435 95.885 0))
     (property "Value" "4k7" (id 1) (at 179.07 97.79 0))
-    (property "Footprint" "Resistor_SMD:R_0603_1608Metric" (id 2) (at 175.895 96.52 0)
+    (property "Footprint" "Resistor_SMD:R_0402_1005Metric" (id 2) (at 175.895 96.52 0)
       (effects (font (size 1.27 1.27)) hide)
     )
@@
       (effects (font (size 1.27 1.27)) (justify left))
     )
-    (property "Footprint" "" (id 2) (at 268.605 33.02 0)
+    (property "Footprint" "Capacitor_SMD:C_0402_1005Metric" (id 2) (at 268.605 33.02 0)
       (effects (font (size 1.27 1.27)) hide)
     )
@@
     (property "Reference" "R?" (id 0) (at 33.655 160.02 90))
     (property "Value" "10k" (id 1) (at 33.655 161.925 90))
-    (property "Footprint" "" (id 2) (at 33.655 163.83 0)
+    (property "Footprint" "Resistor_SMD:R_0402_1005Metric" (id 2) (at 33.655 163.83 0)
       (effects (font (size 1.27 1.27)) hide)
     )
@@
       (effects (font (size 1.27 1.27)) (justify left))
     )
-    (property "Footprint" "" (id 2) (at 138.43 59.69 0)
+    (property "Footprint" "Capacitor_SMD:C_0603_1608Metric" (id 2) (at 138.43 59.69 0)
       (effects (font (size 1.27 1.27)) hide)
     )
@@
       (effects (font (size 1.27 1.27)) (justify left))
     )
-    (property "Footprint" "" (id 2) (at 40.64 34.29 0)
+    (property "Footprint" "Capacitor_SMD:C_0402_1005Metric" (id 2) (at 40.64 34.29 0)
       (effects (font (size 1.27 1.27)) hide)
     )
@@
     (property "Reference" "R?" (id 0) (at 113.03 106.045 90))
     (property "Value" "1k" (id 1) (at 113.03 109.855 90))
-    (property "Footprint" "Resistor_SMD:R_0603_1608Metric" (id 2) (at 113.03 107.95 0)
+    (property "Footprint" "Resistor_SMD:R_0402_1005Metric" (id 2) (at 113.03 107.95 0)
       (effects (font (size 1.27 1.27)) hide)
     )
@@
     (property "Reference" "FB?" (id 0) (at 125.73 24.13 90))
     (property "Value" "100@100MHz" (id 1) (at 125.73 26.035 90))
-    (property "Footprint" "" (id 2) (at 125.73 27.432 90)
+    (property "Footprint" "Inductor_SMD:L_0603_1608Metric" (id 2) (at 125.73 27.432 90)
       (effects (font (size 1.27 1.27)) hide)
     )
@@
     (property "Reference" "R?" (id 0) (at 168.275 95.885 0))
     (property "Value" "4k7" (id 1) (at 168.91 97.79 0))
-    (property "Footprint" "Resistor_SMD:R_0603_1608Metric" (id 2) (at 165.735 96.52 0)
+    (property "Footprint" "Resistor_SMD:R_0402_1005Metric" (id 2) (at 165.735 96.52 0)
       (effects (font (size 1.27 1.27)) hide)
     )
@@
       (effects (font (size 1.27 1.27)) (justify left))
     )
-    (property "Footprint" "" (id 2) (at 112.395 35.56 0)
+    (property "Footprint" "Capacitor_SMD:C_0402_1005Metric" (id 2) (at 112.395 35.56 0)
       (effects (font (size 1.27 1.27)) hide)
     )
@@
     (property "Reference" "R?" (id 0) (at 210.82 95.885 0))
     (property "Value" "4k7" (id 1) (at 211.455 97.79 0))
-    (property "Footprint" "Resistor_SMD:R_0603_1608Metric" (id 2) (at 208.28 96.52 0)
+    (property "Footprint" "Resistor_SMD:R_0402_1005Metric" (id 2) (at 208.28 96.52 0)
       (effects (font (size 1.27 1.27)) hide)
     )
@@
     (property "Reference" "R?" (id 0) (at 187.96 95.885 0))
     (property "Value" "4k7" (id 1) (at 188.595 97.79 0))
-    (property "Footprint" "Resistor_SMD:R_0603_1608Metric" (id 2) (at 185.42 96.52 0)
+    (property "Footprint" "Resistor_SMD:R_0402_1005Metric" (id 2) (at 185.42 96.52 0)
       (effects (font (size 1.27 1.27)) hide)
     )
@@
       (effects (font (size 1.27 1.27)) (justify left))
     )
-    (property "Footprint" "Resistor_SMD:R_0603_1608Metric" (id 2) (at 106.045 103.505 0)
+    (property "Footprint" "Resistor_SMD:R_0402_1005Metric" (id 2) (at 106.045 103.505 0)
       (effects (font (size 1.27 1.27)) hide)
     )
@@
       (effects (font (size 1.27 1.27)) (justify left))
     )
-    (property "Footprint" "" (id 2) (at 102.87 35.56 0)
+    (property "Footprint" "Capacitor_SMD:C_0402_1005Metric" (id 2) (at 102.87 35.56 0)
       (effects (font (size 1.27 1.27)) hide)
     )
@@
       (effects (font (size 1.27 1.27)) (justify left))
     )
-    (property "Footprint" "" (id 2) (at 174.625 28.575 0)
+    (property "Footprint" "Capacitor_SMD:C_0402_1005Metric" (id 2) (at 174.625 28.575 0)
       (effects (font (size 1.27 1.27)) hide)
     )
@@
       (effects (font (size 1.27 1.27)) (justify right))
     )
-    (property "Footprint" "" (id 2) (at 145.415 143.51 90)
+    (property "Footprint" "LED_SMD:LED_0603_1608Metric" (id 2) (at 145.415 143.51 90)
       (effects (font (size 1.27 1.27)) hide)
     )
@@
     (property "Reference" "R?" (id 0) (at 125.73 106.045 90))
     (property "Value" "1k" (id 1) (at 125.73 109.855 90))
-    (property "Footprint" "Resistor_SMD:R_0603_1608Metric" (id 2) (at 125.73 107.95 0)
+    (property "Footprint" "Resistor_SMD:R_0402_1005Metric" (id 2) (at 125.73 107.95 0)
       (effects (font (size 1.27 1.27)) hide)
     )
@@
       (effects (font (size 1.27 1.27)) (justify right))
     )
-    (property "Footprint" "" (id 2) (at 130.175 143.51 90)
+    (property "Footprint" "LED_SMD:LED_0603_1608Metric" (id 2) (at 130.175 143.51 90)
       (effects (font (size 1.27 1.27)) hide)
     )
@@
       (effects (font (size 1.27 1.27)) (justify left))
     )
-    (property "Footprint" "" (id 2) (at 78.105 67.945 0)
+    (property "Footprint" "Capacitor_SMD:C_0402_1005Metric" (id 2) (at 78.105 67.945 0)
       (effects (font (size 1.27 1.27)) hide)
     )
@@
       (effects (font (size 1.27 1.27)) (justify left))
     )
-    (property "Footprint" "" (id 2) (at 31.115 34.29 0)
+    (property "Footprint" "Capacitor_SMD:C_0402_1005Metric" (id 2) (at 31.115 34.29 0)
       (effects (font (size 1.27 1.27)) hide)
     )
@@
       (effects (font (size 1.27 1.27)) (justify left))
     )
-    (property "Footprint" "" (id 2) (at 20.955 34.29 0)
+    (property "Footprint" "Capacitor_SMD:C_0603_1608Metric" (id 2) (at 20.955 34.29 0)
       (effects (font (size 1.27 1.27)) hide)
     )
@@
     (property "Reference" "R?" (id 0) (at 196.215 95.885 0))
     (property "Value" "4k7" (id 1) (at 196.85 97.79 0))
-    (property "Footprint" "Resistor_SMD:R_0603_1608Metric" (id 2) (at 193.675 96.52 0)
+    (property "Footprint" "Resistor_SMD:R_0402_1005Metric" (id 2) (at 193.675 96.52 0)
       (effects (font (size 1.27 1.27)) hide)
     )
@@
       (effects (font (size 1.27 1.27)) (justify left))
     )
-    (property "Footprint" "" (id 2) (at 68.58 67.945 0)
+    (property "Footprint" "Capacitor_SMD:C_0402_1005Metric" (id 2) (at 68.58 67.945 0)
       (effects (font (size 1.27 1.27)) hide)
     )
@@
       (effects (font (size 1.27 1.27)) (justify left))
     )
-    (property "Footprint" "Resistor_SMD:R_0603_1608Metric" (id 2) (at 106.045 112.395 0)
+    (property "Footprint" "Resistor_SMD:R_0402_1005Metric" (id 2) (at 106.045 112.395 0)
       (effects (font (size 1.27 1.27)) hide)
     )
@@
       (effects (font (size 1.27 1.27)) (justify left))
     )
-    (property "Footprint" "" (id 2) (at 119.38 113.665 0)
-      (effects (font (size 1.27 1.27)) hide)
-    )
+    (property "Footprint" "Capacitor_SMD:C_0603_1608Metric" (id 2) (at 119.38 113.665 0)
+      (effects (font (size 1.27 1.27)) hide)
+    )
